File: christmas-ornament.kicad_pcb (KiCad board)
At the start: 2 copper layers, 35.6 x 35.6 mm, 20 parts, among them SW1 SW_SPDT

Commit message: stencil!
Parts:
- removed D4, D6: LED, salvation:LED_1206_ReverseMountSquare1.5mm_HandSolder
- removed R4: 68, Resistor_SMD:R_0805_2012Metric_Pad1.15x1.40mm_HandSolder
- moved R2 17.6 mm to (149.6, 85.9)
- moved D3 17.0 mm to (159.5, 89.9), turned to 180 degrees
- moved R5 15.8 mm to (165.9, 104.4)
- moved R6 11.5 mm to (176.3, 108.5)
- moved R3 11.4 mm to (155.2, 86.4)
- moved D2 10.6 mm to (145.8, 88.9), turned to 180 degrees
- moved D5 8.84 mm to (166.1, 101.1), turned to 180 degrees
- moved R1 2.34 mm to (140.7, 93.7)
- moved D1 1.52 mm to (138.2, 98.6), turned to 180 degrees
- moved D8 1.02 mm to (143.5, 114.0), turned to 0 degrees
